File: pcbs/control_board_pcb/control_board_pcb.kicad_pcb (KiCad board)
At the start: 4 copper layers, 150 x 130 mm, 13 parts, among them J1 Conn_01x07, J2 Conn_01x07, J3 Conn_01x07, J4 Conn_01x07, J5 Conn_01x02, U1 MT3608, U2 MT3608, U3 MT3608, U4 MT3608, U5 ESP32 WROOM 32D DevKit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

Commit message: Control Board PCB Ready
Parts:
- removed D1: 1N4148WT, Diode_SMD:D_SOD-523
- added D2: B120-E3, Diode_SMD:D_SMA, F.Cu at (59.5, 50.0)
- added J6: Conn_01x03, Connector_JST:JST_XH_B3B-XH-A_1x03_P2.50mm_Vertical, F.Cu at (174.5, 76.0)
- added J7: Conn_01x03, Connector_JST:JST_XH_B3B-XH-A_1x03_P2.50mm_Vertical, F.Cu at (174.5, 89.5)
Connections:
- U5 pad 10: unconnected-(U5-D27-Pad10) -> /EN_3
- U5 pad 11: unconnected-(U5-D14-Pad11) -> /DIR_3
- U5 pad 12: unconnected-(U5-D12-Pad12) -> /STEP_3
- U5 pad 4: /EN_4 -> unconnected-(U5-D34-Pad4)
- U5 pad 5: /DIR_4 -> /LIMIT_SW_1
- U5 pad 6: /STEP_4 -> /LIMIT_SW_2
- U5 pad 7: /EN_3 -> /EN_4
- U5 pad 8: /DIR_3 -> /DIR_4
- U5 pad 9: /STEP_3 -> /STEP_4
Routing:
- net /LIMIT_SW_2: track 0.00 -> 121.1 mm
- net /LIMIT_SW_1: track 0.00 -> 106.0 mm
- net /STEP_3: track 178.7 -> 195.4 mm
- net /DIR_3: track 172.4 -> 188.9 mm
- net /EN_3: track 166.1 -> 182.5 mm
- net /STEP_4: track 143.8 -> 160.0 mm
- net /DIR_4: track 137.5 -> 153.6 mm
- net /EN_4: track 131.5 -> 147.4 mm
- net +5V: track 27.2 -> 25.7 mm
- net +24V_1: track 41.8 -> 43.3 mm
- net +24V_2: track 41.5 -> 42.8 mm
- net +24V_4: track 39.2 -> 40.1 mm
- net /EN_1: track 119.6 -> 118.9 mm, vias 0 -> 1
- net /STEP_1: track 121.3 -> 120.6 mm, vias 0 -> 1
- net /DIR_1: track 120.2 -> 119.7 mm, vias 0 -> 1
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
Commit message: Motor Controller Interface almost ready
Parts:
- added REF**: MountingHole_3.2mm_M3, MountingHole:MountingHole_3.2mm_M3, F.Cu at (40.0, 155.0)
- added REF**: MountingHole_3.2mm_M3, MountingHole:MountingHole_3.2mm_M3, F.Cu at (180.0, 155.0)
- added REF**: MountingHole_3.2mm_M3, MountingHole:MountingHole_3.2mm_M3, F.Cu at (40.0, 35.0)
- added REF**: MountingHole_3.2mm_M3, MountingHole:MountingHole_3.2mm_M3, F.Cu at (180.0, 34.5)
- moved U6 6.53 mm to (80.0, 120.0)
Routing:
- net +5V: track 25.7 -> 28.4 mm
- net /EN_2: track 135.7 -> 138.1 mm
- net /EN_1: track 118.9 -> 121.2 mm
- net /DIR_2: track 135.6 -> 138.0 mm
- net /STEP_1: track 120.6 -> 122.9 mm
- net /DIR_1: track 119.7 -> 122.0 mm
- net /STEP_2: track 135.5 -> 137.8 mm

Commit message: Order PCBs
Connections:
- J6 pad 2: +3V3 -> GND
- J6 pad 3: GND -> +3V3
- J7 pad 2: +3V3 -> GND
- J7 pad 3: GND -> +3V3
Changed lines of the file:
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@@
 			(outputformat 1)
 			(mirror no)
-			(drillshape 1)
+			(drillshape 0)
 			(scaleselection 1)
-			(outputdirectory "")
+			(outputdirectory "export/")
 		)
 	)
@@
 			(layers "*.Cu" "*.Mask")
 			(remove_unused_layers no)
-			(net 18 "+3V3")
+			(net 14 "GND")
 			(pinfunction "Pin_2")
 			(pintype "passive")
@@
 			(layers "*.Cu" "*.Mask")
 			(remove_unused_layers no)
-			(net 14 "GND")
+			(net 18 "+3V3")
 			(pinfunction "Pin_3")
 			(pintype "passive")
@@
 			(pintype "input")
 		)
+		(pad "5" thru_hole oval
+			(at 15.24 -1.27 180)
+			(size 1.7 1.7)
+			(drill 1)
+			(layers "*.Cu" "*.Mask")
+			(remove_unused_layers no)
+		)
+		(pad "6" thru_hole oval
+			(at 15.24 1.27 180)
+			(size 1.7 1.7)
+			(drill 1)
+			(layers "*.Cu" "*.Mask")
+			(remove_unused_layers no)
+		)
+		(pad "7" thru_hole oval
+			(at -15.24 -1.27 180)
+			(size 1.7 1.7)
+			(drill 1)
+			(layers "*.Cu" "*.Mask")
+			(remove_unused_layers no)
+		)
+		(pad "8" thru_hole oval
+			(at -15.24 1.27 180)
+			(size 1.7 1.7)
+			(drill 1)
+			(layers "*.Cu" "*.Mask")
+			(remove_unused_layers no)
+		)
 		(embedded_fonts no)
 	)
@@
 			(pintype "input")
 		)
+		(pad "5" thru_hole oval
+			(at 15.24 -1.27 180)
+			(size 1.7 1.7)
+			(drill 1)
+			(layers "*.Cu" "*.Mask")
+			(remove_unused_layers no)
+		)
+		(pad "6" thru_hole oval
+			(at 15.24 1.27 180)
+			(size 1.7 1.7)
+			(drill 1)
+			(layers "*.Cu" "*.Mask")
+			(remove_unused_layers no)
+		)
+		(pad "7" thru_hole oval
+			(at -15.24 -1.27 180)
+			(size 1.7 1.7)
+			(drill 1)
+			(layers "*.Cu" "*.Mask")
+			(remove_unused_layers no)
+		)
+		(pad "8" thru_hole oval
+			(at -15.24 1.27 180)
+			(size 1.7 1.7)
+			(drill 1)
+			(layers "*.Cu" "*.Mask")
+			(remove_unused_layers no)
+		)
 		(embedded_fonts no)
 	)
@@
 			(pintype "input")
 		)
+		(pad "5" thru_hole oval
+			(at 15.24 -1.27 180)
+			(size 1.7 1.7)
+			(drill 1)
+			(layers "*.Cu" "*.Mask")
+			(remove_unused_layers no)
+		)
+		(pad "6" thru_hole oval
+			(at 15.24 1.27 180)
+			(size 1.7 1.7)
+			(drill 1)
+			(layers "*.Cu" "*.Mask")
+			(remove_unused_layers no)
+		)
+		(pad "7" thru_hole oval
+			(at -15.24 -1.27 180)
+			(size 1.7 1.7)
+			(drill 1)
+			(layers "*.Cu" "*.Mask")
+			(remove_unused_layers no)
+		)
+		(pad "8" thru_hole oval
+			(at -15.24 1.27 180)
+			(size 1.7 1.7)
+			(drill 1)
+			(layers "*.Cu" "*.Mask")
+			(remove_unused_layers no)
+		)
 		(embedded_fonts no)
 	)
@@
 			(pintype "input")
 		)
+		(pad "5" thru_hole oval
+			(at 15.24 -1.27 180)
+			(size 1.7 1.7)
+			(drill 1)
+			(layers "*.Cu" "*.Mask")
+			(remove_unused_layers no)
+		)
+		(pad "6" thru_hole oval
+			(at 15.24 1.27 180)
+			(size 1.7 1.7)
+			(drill 1)
+			(layers "*.Cu" "*.Mask")
+			(remove_unused_layers no)
+		)
+		(pad "7" thru_hole oval
+			(at -15.24 -1.27 180)
+			(size 1.7 1.7)
+			(drill 1)
+			(layers "*.Cu" "*.Mask")
+			(remove_unused_layers no)
+		)
+		(pad "8" thru_hole oval
+			(at -15.24 1.27 180)
+			(size 1.7 1.7)
+			(drill 1)
+			(layers "*.Cu" "*.Mask")
+			(remove_unused_layers no)
+		)
 		(embedded_fonts no)
 	)
@@
 			(layers "*.Cu" "*.Mask")
 			(remove_unused_layers no)
-			(net 18 "+3V3")
+			(net 14 "GND")
 			(pinfunction "Pin_2")
 			(pintype "passive")
@@
 			(layers "*.Cu" "*.Mask")
 			(remove_unused_layers no)
-			(net 14 "GND")
+			(net 18 "+3V3")
 			(pinfunction "Pin_3")
 			(pintype "passive")
