File: pcbs/control_board_pcb/control_board_pcb.kicad_sch (KiCad schematic)
At the start: 5 parts, among them U1 MT3608, U2 MT3608, U3 MT3608, U4 MT3608, U5 ESP32 WROOM 32D DevKit

Commit message: Control PCB nearly complete
Parts:
- added D1: 1N4148WT, Diode_SMD:D_SOD-523, symbol Diode:1N4148WT
- added J1, J2, J3, J4: Conn_01x07, Connector_JST:JST_XH_B7B-XH-A_1x07_P2.50mm_Vertical, symbol Connector_Generic:Conn_01x07
- added J5: Conn_01x02, Connector_PinHeader_2.54mm:PinHeader_1x02_P2.54mm_Vertical, symbol Connector_Generic:Conn_01x02
- added U6: HU-M28, control_board_pcb:HU-M28, symbol control_board_pcb:HU-M28
- added U7: DSN-VC288, control_board_pcb:DSN-VC228_Pin-Holes, symbol control_board_pcb:DSN-VS228_Pin-Holes
Connections:
- net +12V: now also U6.3 (12V), U7.1 (VCC), U7.2 (Supply_V)
- net GND: now also U5.14 (GND), U5.17 (GND), J1.6 (Pin_6), J1.7 (Pin_7), J2.6 (Pin_6), J2.7 (Pin_7), J3.6 (Pin_6), J3.7 (Pin_7), J4.6 (Pin_6), J4.7 (Pin_7), J5.2 (Pin_2), U7.3 (Shunt_Load_Neg)
- net at U5.15 (VIN): now also D1.1 (K)
- net +3V3: now reaches U5.16 (3V3)
- net +3V3: now also J1.2 (Pin_2), J2.2 (Pin_2), J3.2 (Pin_2), J4.2 (Pin_2)
- net STEP_1: now reaches U5.21 (D16)
- net STEP_1: now also J1.3 (Pin_3)
- net DIR_1: now reaches U5.22 (D17)
- net DIR_1: now also J1.4 (Pin_4)
- net EN_1: now reaches U5.23 (D5)
- net EN_1: now also J1.5 (Pin_5)
- net STEP_2: now reaches U5.24 (D18)
- net STEP_2: now also J2.3 (Pin_3)
- net DIR_2: now reaches U5.25 (D19)
- net DIR_2: now also J2.4 (Pin_4)
- net EN_2: now reaches U5.26 (D21)
- net EN_2: now also J2.5 (Pin_5)
- net EN_4: now reaches U5.4 (D34)
- net EN_4: now also J4.5 (Pin_5)
- net DIR_4: now reaches U5.5 (D35)
- net DIR_4: now also J4.4 (Pin_4)
- net STEP_4: now reaches U5.6 (D32)
- net STEP_4: now also J4.3 (Pin_3)
- net EN_3: now reaches U5.7 (D33)
- net EN_3: now also J3.5 (Pin_5)
- net DIR_3: now reaches U5.8 (D25)
- net DIR_3: now also J3.4 (Pin_4)
- net STEP_3: now reaches U5.9 (D26)
- net STEP_3: now also J3.3 (Pin_3)
- removed net +24V1: U1.3 (VOUT+), U2.3 (VOUT+), U3.3 (VOUT+), U4.3 (VOUT+)
- new net +24V_1: J1.1 (Pin_1), U1.3 (VOUT+)
- new net +24V_2: J2.1 (Pin_1), U2.3 (VOUT+)
- new net +24V_3: J3.1 (Pin_1), U3.3 (VOUT+)
- new net +24V_4: J4.1 (Pin_1), U4.3 (VOUT+)
- new net +3V3_PSU: U6.7 (3V3)
- new net +5V: D1.2 (A), U6.5 (5V)
- new net -12V: U6.1 (-12V)
- new net GND_PSU: J5.1 (Pin_1), U6.2 (GND), U6.4 (GND), U6.6 (GND), U6.8 (GND), U7.4 (Shunt_GND), U7.5 (GND)
Other:
- moved on the sheet: U1, U2, U3, U4, U5

Commit message: Control Board PCB Ready
Parts:
- removed D1: 1N4148WT, Diode_SMD:D_SOD-523, symbol Diode:1N4148WT
- added D2: B120-E3, Diode_SMD:D_SMA, symbol Diode:B120-E3
- added J6, J7: Conn_01x03, Connector_JST:JST_XH_B3B-XH-A_1x03_P2.50mm_Vertical, symbol Connector_Generic:Conn_01x03
Connections:
- net +3V3: now also J6.2 (Pin_2), J7.2 (Pin_2)
- net +5V: now also D2.2 (A)
- net DIR_3: now also U5.11 (D14); no longer U5.8 (D25)
- net DIR_4: now also U5.8 (D25); no longer U5.5 (D35)
- net EN_3: now also U5.10 (D27); no longer U5.7 (D33)
- net EN_4: now also U5.7 (D33); no longer U5.4 (D34)
- net GND: now also J6.3 (Pin_3), J7.3 (Pin_3)
- net STEP_3: now also U5.12 (D12); no longer U5.9 (D26)
- net STEP_4: now also U5.9 (D26); no longer U5.6 (D32)
- net at U5.15 (VIN): now also D2.1 (K)
- new net LIMIT_SW_1: J6.1 (Pin_1), U5.5 (D35)
- new net LIMIT_SW_2: J7.1 (Pin_1), U5.6 (D32)

Commit message: Order PCBs
Connections:
- net +3V3: now also J6.3 (Pin_3), J7.3 (Pin_3); no longer J6.2 (Pin_2), J7.2 (Pin_2)
- net GND: now also J6.2 (Pin_2), J7.2 (Pin_2); no longer J6.3 (Pin_3), J7.3 (Pin_3)
Changed lines of the file:
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@@
 	(wire
 		(pts
-			(xy 228.6 113.03) (xy 242.57 113.03)
+			(xy 115.57 58.42) (xy 116.84 58.42)
 		)
 		(stroke
@@
 	(wire
 		(pts
-			(xy 115.57 58.42) (xy 116.84 58.42)
+			(xy 142.24 74.93) (xy 143.51 74.93)
 		)
 		(stroke
@@
 	(wire
 		(pts
-			(xy 142.24 74.93) (xy 143.51 74.93)
+			(xy 115.57 83.82) (xy 116.84 83.82)
 		)
 		(stroke
@@
 	(wire
 		(pts
-			(xy 115.57 83.82) (xy 116.84 83.82)
+			(xy 228.6 107.95) (xy 242.57 107.95)
 		)
 		(stroke
@@
 	(wire
 		(pts
-			(xy 228.6 133.35) (xy 242.57 133.35)
-		)
-		(stroke
-			(width 0)
-			(type default)
-		)
-	)
-	(wire
-		(pts
 			(xy 93.98 104.14) (xy 95.25 104.14)
 		)
@@
 	(wire
 		(pts
-			(xy 228.6 130.81) (xy 242.57 130.81)
-		)
-		(stroke
-			(width 0)
-			(type default)
-		)
-	)
-	(wire
-		(pts
 			(xy 201.93 62.23) (xy 203.2 62.23)
 		)
@@
 	(wire
 		(pts
+			(xy 228.6 110.49) (xy 242.57 110.49)
+		)
+		(stroke
+			(width 0)
+			(type default)
+		)
+	)
+	(wire
+		(pts
 			(xy 115.57 53.34) (xy 116.84 53.34)
 		)
@@
 	(wire
 		(pts
+			(xy 228.6 128.27) (xy 242.57 128.27)
+		)
+		(stroke
+			(width 0)
+			(type default)
+		)
+	)
+	(wire
+		(pts
 			(xy 201.93 72.39) (xy 203.2 72.39)
 		)
@@
 	(wire
 		(pts
+			(xy 228.6 130.81) (xy 242.57 130.81)
+		)
+		(stroke
+			(width 0)
+			(type default)
+		)
+	)
+	(wire
+		(pts
 			(xy 93.98 53.34) (xy 95.25 53.34)
 		)
@@
 	(wire
 		(pts
-			(xy 228.6 110.49) (xy 242.57 110.49)
-		)
-		(stroke
-			(width 0)
-			(type default)
-		)
-	)
-	(wire
-		(pts
 			(xy 195.58 118.11) (xy 195.58 120.65)
 		)
@@
 	)
 	(label "LIMIT_SW_1"
-		(at 242.57 107.95 180)
+		(at 242.57 113.03 180)
 		(effects
 			(font
@@
 	)
 	(label "LIMIT_SW_2"
-		(at 242.57 128.27 180)
+		(at 242.57 133.35 180)
 		(effects
 			(font
@@
 	(symbol
 		(lib_id "power:+12V")
-		(at 228.6 110.49 0)
+		(at 228.6 107.95 0)
 		(unit 1)
 		(exclude_from_sim no)
@@
 		(fields_autoplaced yes)
 		(property "Reference" "#PWR021"
-			(at 228.6 114.3 0)
+			(at 228.6 111.76 0)
 			(effects
 				(font
@@
 		)
 		(property "Value" "+3V3"
-			(at 228.6 105.41 0)
+			(at 228.6 102.87 0)
 			(effects
 				(font
@@
 		)
 		(property "Footprint" ""
-			(at 228.6 110.49 0)
+			(at 228.6 107.95 0)
 			(effects
 				(font
@@
 		)
 		(property "Datasheet" ""
-			(at 228.6 110.49 0)
+			(at 228.6 107.95 0)
 			(effects
 				(font
@@
 		)
 		(property "Description" "Power symbol creates a global label with name \"+12V\""
-			(at 228.6 110.49 0)
+			(at 228.6 107.95 0)
 			(effects
 				(font
@@
 		(lib_id "Connector_Generic:Conn_01x03")
 		(at 247.65 110.49 0)
+		(mirror x)
 		(unit 1)
 		(exclude_from_sim no)
@@
 		(on_board yes)
 		(dnp no)
-		(fields_autoplaced yes)
 		(property "Reference" "J6"
-			(at 250.19 109.2199 0)
+			(at 250.19 111.7601 0)
 			(effects
 				(font
@@
 		)
 		(property "Value" "Conn_01x03"
-			(at 250.19 111.7599 0)
+			(at 250.19 109.2201 0)
 			(effects
 				(font
@@
 	(symbol
 		(lib_id "power:GND")
-		(at 228.6 133.35 0)
+		(at 228.6 130.81 0)
 		(unit 1)
 		(exclude_from_sim no)
@@
 		(fields_autoplaced yes)
 		(property "Reference" "#PWR024"
-			(at 228.6 139.7 0)
+			(at 228.6 137.16 0)
 			(effects
 				(font
@@
 		)
 		(property "Value" "GND"
-			(at 228.6 138.43 0)
+			(at 228.6 135.89 0)
 			(effects
 				(font
@@
 		)
 		(property "Footprint" ""
-			(at 228.6 133.35 0)
+			(at 228.6 130.81 0)
 			(effects
 				(font
@@
 		)
 		(property "Datasheet" ""
-			(at 228.6 133.35 0)
+			(at 228.6 130.81 0)
 			(effects
 				(font
@@
 		)
 		(property "Description" "Power symbol creates a global label with name \"GND\" , ground"
-			(at 228.6 133.35 0)
+			(at 228.6 130.81 0)
 			(effects
 				(font
@@
 	(symbol
 		(lib_id "power:+12V")
-		(at 228.6 130.81 0)
+		(at 228.6 128.27 0)
 		(unit 1)
 		(exclude_from_sim no)
@@
 		(fields_autoplaced yes)
 		(property "Reference" "#PWR023"
-			(at 228.6 134.62 0)
+			(at 228.6 132.08 0)
 			(effects
 				(font
@@
 		)
 		(property "Value" "+3V3"
-			(at 228.6 125.73 0)
+			(at 228.6 123.19 0)
 			(effects
 				(font
@@
 		)
 		(property "Footprint" ""
-			(at 228.6 130.81 0)
+			(at 228.6 128.27 0)
 			(effects
 				(font
@@
 		)
 		(property "Datasheet" ""
-			(at 228.6 130.81 0)
+			(at 228.6 128.27 0)
 			(effects
 				(font
@@
 		)
 		(property "Description" "Power symbol creates a global label with name \"+12V\""
-			(at 228.6 130.81 0)
+			(at 228.6 128.27 0)
 			(effects
 				(font
@@
 	(symbol
 		(lib_id "power:GND")
-		(at 228.6 113.03 0)
+		(at 228.6 110.49 0)
 		(unit 1)
 		(exclude_from_sim no)
@@
 		(fields_autoplaced yes)
 		(property "Reference" "#PWR020"
-			(at 228.6 119.38 0)
+			(at 228.6 116.84 0)
 			(effects
 				(font
@@
 		)
 		(property "Value" "GND"
-			(at 228.6 118.11 0)
+			(at 228.6 115.57 0)
 			(effects
 				(font
@@
 		)
 		(property "Footprint" ""
-			(at 228.6 113.03 0)
+			(at 228.6 110.49 0)
 			(effects
 				(font
@@
 		)
 		(property "Datasheet" ""
-			(at 228.6 113.03 0)
+			(at 228.6 110.49 0)
 			(effects
 				(font
@@
 		)
 		(property "Description" "Power symbol creates a global label with name \"GND\" , ground"
-			(at 228.6 113.03 0)
+			(at 228.6 110.49 0)
 			(effects
 				(font
@@
 		(lib_id "Connector_Generic:Conn_01x03")
 		(at 247.65 130.81 0)
+		(mirror x)
 		(unit 1)
 		(exclude_from_sim no)
@@
 		(on_board yes)
 		(dnp no)
-		(fields_autoplaced yes)
 		(property "Reference" "J7"
-			(at 250.19 129.5399 0)
+			(at 250.19 132.0801 0)
 			(effects
 				(font
@@
 		)
 		(property "Value" "Conn_01x03"
-			(at 250.19 132.0799 0)
+			(at 250.19 129.5401 0)
 			(effects
 				(font
